File: _autosave-flightcomputerv1.kicad_sch (KiCad schematic)
At the start: 51 parts, among them IC1 MMC5983MA, J1 Screw_Terminal_01x02, J2 Screw_Terminal_01x02, J5 Conn_01x02, J6 Conn_01x24, J7 Conn_01x24, J8 Conn_Coaxial, J9 Conn_Coaxial, M1 Motor_Servo, M2 Motor_Servo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

Commit message: finished most of routing 2/28
Connections:
- net radio_cs: now also J6.20 (Pin_20), U1.20 (28_RX7); no longer J6.24 (Pin_24), U1.24 (32_OUT1B)
- net radio_dio5: now also J6.24 (Pin_24), U1.24 (32_OUT1B); no longer J6.20 (Pin_20), U1.20 (28_RX7)
Changed lines of the file:
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@@
 	(wire
 		(pts
+			(xy 157.48 121.92) (xy 170.18 121.92)
+		)
+		(stroke
+			(width 0)
+			(type default)
+		)
+	)
+	(wire
+		(pts
 			(xy 190.5 38.1) (xy 194.31 38.1)
 		)
@@
 	(wire
 		(pts
-			(xy 157.48 104.14) (xy 170.18 104.14)
+			(xy 157.48 132.08) (xy 170.18 132.08)
 		)
 		(stroke
@@
 	(wire
 		(pts
-			(xy 270.51 80.01) (xy 283.21 80.01)
+			(xy 157.48 104.14) (xy 170.18 104.14)
 		)
 		(stroke
@@
 	(wire
 		(pts
-			(xy 157.48 132.08) (xy 170.18 132.08)
-		)
-		(stroke
-			(width 0)
-			(type default)
-		)
-	)
-	(wire
-		(pts
 			(xy 171.45 242.57) (xy 182.88 242.57)
 		)
@@
 	(wire
 		(pts
-			(xy 270.51 90.17) (xy 283.21 90.17)
-		)
-		(stroke
-			(width 0)
-			(type default)
-		)
-	)
-	(wire
-		(pts
 			(xy 154.94 38.1) (xy 160.02 38.1)
 		)
@@
 	(wire
 		(pts
-			(xy 157.48 121.92) (xy 170.18 121.92)
-		)
-		(stroke
-			(width 0)
-			(type default)
-		)
-	)
-	(wire
-		(pts
 			(xy 270.51 82.55) (xy 283.21 82.55)
 		)
@@
 	(wire
 		(pts
+			(xy 270.51 80.01) (xy 283.21 80.01)
+		)
+		(stroke
+			(width 0)
+			(type default)
+		)
+	)
+	(wire
+		(pts
 			(xy 394.97 168.91) (xy 394.97 166.37)
 		)
@@
 	(wire
 		(pts
+			(xy 270.51 90.17) (xy 283.21 90.17)
+		)
+		(stroke
+			(width 0)
+			(type default)
+		)
+	)
+	(wire
+		(pts
 			(xy 226.06 81.28) (xy 240.03 81.28)
 		)
@@
 	)
 	(label "radio_cs"
-		(at 157.48 132.08 0)
+		(at 157.48 121.92 0)
 		(fields_autoplaced yes)
 		(effects
@@
 	)
 	(label "radio_dio5"
-		(at 157.48 121.92 0)
+		(at 157.48 132.08 0)
 		(fields_autoplaced yes)
 		(effects
@@
 	)
 	(label "radio_dio5"
-		(at 270.51 80.01 0)
+		(at 270.51 90.17 0)
 		(fields_autoplaced yes)
 		(effects
@@
 	)
 	(label "radio_cs"
-		(at 270.51 90.17 0)
+		(at 270.51 80.01 0)
 		(fields_autoplaced yes)
 		(effects

Commit message: prelim routing placement done 3/2 need to check batt connector footprints + antenna connector + backup radio
Parts:
- M1, M2: footprint Connector_PinHeader_2.54mm:PinHeader_1x03_P2.54mm_Horizontal -> Connector_PinHeader_2.54mm:PinHeader_1x03_P2.54mm_Vertical
Connections:
- net FREE11: now also J6.7 (Pin_7), U1.7 (5_IN2); no longer J6.4 (Pin_4), U1.4 (2_OUT2)
- net FREE12: now also J6.8 (Pin_8), U1.8 (6_OUT1D); no longer J6.5 (Pin_5), U1.5 (3_LRCLK2)
- net FREE6: now also J7.7 (Pin_7), U1.31 (39_MISO1_OUT1A); no longer J6.6 (Pin_6), U1.6 (4_BCLK2)
- net LED1: now also J6.6 (Pin_6), U1.6 (4_BCLK2); no longer J7.9 (Pin_9), U1.33 (41_A17)
- net LED2: now also J6.5 (Pin_5), U1.5 (3_LRCLK2); no longer J7.8 (Pin_8), U1.32 (40_A16)
- net LED3: now also J6.4 (Pin_4), U1.4 (2_OUT2); no longer J7.7 (Pin_7), U1.31 (39_MISO1_OUT1A)
- net PYRO1: now also J7.8 (Pin_8), U1.32 (40_A16); no longer J7.12 (Pin_12), U1.36 (14_A0_TX3_SPDIF_OUT)
- net PYRO2: now also J7.9 (Pin_9), U1.33 (41_A17); no longer J7.13 (Pin_13), U1.37 (15_A1_RX3_SPDIF_IN)
- net servo1_pwm: now also J7.13 (Pin_13), U1.37 (15_A1_RX3_SPDIF_IN); no longer J6.8 (Pin_8), U1.8 (6_OUT1D)
- net servo2_pwm: now also J7.12 (Pin_12), U1.36 (14_A0_TX3_SPDIF_OUT); no longer J6.7 (Pin_7), U1.7 (5_IN2)
