File: flightcomputerv1.kicad_sch (KiCad schematic)
At the start: 51 parts, among them IC1 MMC5983MA, J1 Screw_Terminal_01x02, J2 Screw_Terminal_01x02, J5 Conn_01x02, J6 Conn_01x24, J7 Conn_01x24, J8 Conn_Coaxial, J9 Conn_Coaxial, M1 Motor_Servo, M2 Motor_Servo, Q1 SI4925DDY-T1-GE3, Q2 MMBT3904, Q3 MMBT3904, SW2 SW_Wuerth_450301014042, U1 Teensy4.1, U2 MS5607-02BA, U3 BMI088, U4 MIC29302AWD, U5 MAX-M10S, U6 RFM95W-915S2, U7 LD1117S50TR_SOT223

Commit message: prelim routing placement done 3/2 need to check batt connector footprints + antenna connector + backup radio
Connections:
- net FREE11: now also J6.7 (Pin_7), U1.7 (5_IN2); no longer J6.4 (Pin_4), U1.4 (2_OUT2)
- net FREE12: now also J6.8 (Pin_8), U1.8 (6_OUT1D); no longer J6.5 (Pin_5), U1.5 (3_LRCLK2)
- net FREE6: now also J7.7 (Pin_7), U1.31 (39_MISO1_OUT1A); no longer J6.6 (Pin_6), U1.6 (4_BCLK2)
- net LED1: now also J6.6 (Pin_6), U1.6 (4_BCLK2); no longer J7.9 (Pin_9), U1.33 (41_A17)
- net LED2: now also J6.5 (Pin_5), U1.5 (3_LRCLK2); no longer J7.8 (Pin_8), U1.32 (40_A16)
- net LED3: now also J6.4 (Pin_4), U1.4 (2_OUT2); no longer J7.7 (Pin_7), U1.31 (39_MISO1_OUT1A)
- net PYRO1: now also J7.8 (Pin_8), U1.32 (40_A16); no longer J7.12 (Pin_12), U1.36 (14_A0_TX3_SPDIF_OUT)
- net PYRO2: now also J7.9 (Pin_9), U1.33 (41_A17); no longer J7.13 (Pin_13), U1.37 (15_A1_RX3_SPDIF_IN)
- net radio_cs: now also J6.20 (Pin_20), U1.20 (28_RX7); no longer J6.24 (Pin_24), U1.24 (32_OUT1B)
- net radio_dio5: now also J6.24 (Pin_24), U1.24 (32_OUT1B); no longer J6.20 (Pin_20), U1.20 (28_RX7)
- net servo1_pwm: now also J7.13 (Pin_13), U1.37 (15_A1_RX3_SPDIF_IN); no longer J6.8 (Pin_8), U1.8 (6_OUT1D)
- net servo2_pwm: now also J7.12 (Pin_12), U1.36 (14_A0_TX3_SPDIF_OUT); no longer J6.7 (Pin_7), U1.7 (5_IN2)

Commit message: moved buttons
Parts:
- removed SW2: SW_Wuerth_450301014042, Button_Switch_THT:SW_Slide-03_Wuerth-WS-SLTV_10x2.5x6.4_P2.54mm, symbol Switch:SW_Wuerth_450301014042
- added S2: TS04-66-70-BK-160-SMT, HPRfootprints:SW_TS04-66-70-BK-160-SMT, symbol HPRsymbols:TS04-66-70-BK-160-SMT
- added TP1, TP2, TP3: TestPoint, Connector_PinHeader_2.54mm:PinHeader_1x01_P2.54mm_Vertical, symbol Connector:TestPoint
- M1, M2: footprint Connector_PinHeader_2.54mm:PinHeader_1x03_P2.54mm_Horizontal -> Connector_PinHeader_2.54mm:PinHeader_1x03_P2.54mm_Vertical
Connections:
- net GND: now also S2.2, S2.4
- net VBATT: now also TP1.1
- net ldo_5v: now also TP2.1
- net ldo_6v: now also TP3.1
- net teensy_3.3v: no longer S1.3
- net teensy_onoff: now also S2.1, S2.3
- net at S1.1, U1.53 (PROGRAM): now also S1.3
Other:
- moved on the sheet: S1

Commit message: magnetometer had wrong footprint. fixed all DRC errors. need to remake gerber
Parts:
- IC1: footprint HPRfootprints:PQFN50P450X300X100-16N -> HPRfootprints:MMC5983MA_MEM
Changed lines of the file:
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@@
 			)
 		)
-		(property "Footprint" "HPRfootprints:PQFN50P450X300X100-16N"
+		(property "Footprint" "HPRfootprints:MMC5983MA_MEM"
 			(at 83.82 249.86 0)
 			(effects

Commit message: still need to fill out BOM doc and get quote for assembly
Parts:
- IC1: MPN (none) -> MMC5983MA; Manufacturer (none) -> MEMSIC; Manufacturer_Name MEMSIC -> (none); Manufacturer_Part_Number MMC5983MA -> (none); Mouser Part Number 438-MMC5983MA -> (none); Package (none) -> 16-VFLGA
- Q1: MPN (none) -> SI4925DDY-T1-GE3; Manufacturer (none) -> Vishay Siliconix; Manufacturer_Name Vishay -> (none); Manufacturer_Part_Number SI4925DDY-T1-GE3 -> (none); Mouser Part Number 781-SI4925DDY-GE3 -> (none); Package (none) -> 8-SOIC (0.154", 3.90mm Width)
- S2: MANUFACTURER CUI Devices -> (none); MPN (none) -> TS04-66-70-BK-160-SMT; Manufacturer (none) -> Same Sky (Formerly CUI Devices); Package (none) -> Gull Wing
- U1: now not fitted
- U2: MPN (none) -> MS560702BA03-50; Manufacturer (none) -> TE Connectivity Measurement Specialties; Package (none) -> 8-SMD
- U3: MF Bosch Sensortec -> (none); MP BMI088 -> (none); MPN (none) -> BMI088; Manufacturer (none) -> Bosch Sensortec; PACKAGE VFLGA-16 Bosch Sensortec -> (none); Package (none) -> 16-VFLGA Module
- U4: MPN (none) -> MIC29302AWD-TR; Manufacturer (none) -> Microchip Technology; Package (none) -> TO-252-6, DPAK (5 Leads + Tab)
- U5: MPN (none) -> MAX-M10S-00B; Manufacturer (none) -> u-blox; Package (none) -> 18-SMD Module
- U6: MPN (none) -> RFM95W-915S2; Manufacturer (none) -> RF Solutions; Package (none) -> 16-SMD Module
- U7: MPN (none) -> LD1117S50TR; Manufacturer (none) -> STMicroelectronics; Package (none) -> TO-261-4, TO-261AA
Changed lines of the file:
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@@
 		(in_bom yes)
 		(on_board yes)
-		(dnp no)
+		(dnp yes)
 		(fields_autoplaced yes)
 		(property "Reference" "U1"
@@
 			)
 		)
+		(property "Manufacturer" "STMicroelectronics"
+			(at 223.52 38.1 0)
+			(effects
+				(font
+					(size 1.27 1.27)
+				)
+				(hide yes)
+			)
+		)
+		(property "MPN" "LD1117S50TR"
+			(at 223.52 38.1 0)
+			(effects
+				(font
+					(size 1.27 1.27)
+				)
+				(hide yes)
+			)
+		)
+		(property "Package" "TO-261-4, TO-261AA"
+			(at 223.52 38.1 0)
+			(effects
+				(font
+					(size 1.27 1.27)
+				)
+				(hide yes)
+			)
+		)
 		(pin "1"
 		)
@@
 			)
 		)
+		(property "Manufacturer" "RF Solutions"
+			(at 195.58 242.57 0)
+			(effects
+				(font
+					(size 1.27 1.27)
+				)
+				(hide yes)
+			)
+		)
+		(property "Package" "16-SMD Module"
+			(at 195.58 242.57 0)
+			(effects
+				(font
+					(size 1.27 1.27)
+				)
+				(hide yes)
+			)
+		)
+		(property "MPN" "RFM95W-915S2"
+			(at 195.58 242.57 0)
+			(effects
+				(font
+					(size 1.27 1.27)
+				)
+				(hide yes)
+			)
+		)
 		(pin "1"
 		)
@@
 			)
 		)
-		(property "Description" ""
+		(property "Description" "SWITCH TACTILE SPST-NO 0.05A 12V"
 			(at 287.02 157.48 0)
 			(effects
@@
 			)
 		)
-		(property "MANUFACTURER" "CUI Devices"
+		(property "Manufacturer" "Same Sky (Formerly CUI Devices)"
 			(at 287.02 157.48 0)
 			(effects
@@
 			)
 		)
+		(property "MPN" "TS04-66-70-BK-160-SMT"
+			(at 287.02 157.48 0)
+			(effects
+				(font
+					(size 1.27 1.27)
+				)
+				(hide yes)
+			)
+		)
+		(property "Package" "Gull Wing"
+			(at 287.02 157.48 0)
+			(effects
+				(font
+					(size 1.27 1.27)
+				)
+				(hide yes)
+			)
+		)
 		(pin "1"
 		)
@@
 			)
 		)
-		(property "Mouser Part Number" "781-SI4925DDY-GE3"
+		(property "MPN" "SI4925DDY-T1-GE3"
 			(at 354.33 709.55 0)
 			(effects
@@
 			)
 		)
-		(property "Manufacturer_Name" "Vishay"
+		(property "Manufacturer" "Vishay Siliconix"
 			(at 354.33 909.55 0)
 			(effects
@@
 			)
 		)
-		(property "Manufacturer_Part_Number" "SI4925DDY-T1-GE3"
-			(at 354.33 1009.55 0)
+		(property "Package" "8-SOIC (0.154\", 3.90mm Width)"
+			(at 332.74 214.63 0)
 			(effects
 				(font
 					(size 1.27 1.27)
 				)
-				(justify left top)
 				(hide yes)
 			)
@@
 			)
 		)
+		(property "Package" "8-SMD"
+			(at 87.63 48.26 0)
+			(effects
+				(font
+					(size 1.27 1.27)
+				)
+				(hide yes)
+			)
+		)
+		(property "Manufacturer" "TE Connectivity Measurement Specialties"
+			(at 87.63 48.26 0)
+			(effects
+				(font
+					(size 1.27 1.27)
+				)
+				(hide yes)
+			)
+		)
+		(property "MPN" "MS560702BA03-50"
+			(at 87.63 48.26 0)
+			(effects
+				(font
+					(size 1.27 1.27)
+				)
+				(hide yes)
+			)
+		)
 		(pin "6"
 		)
@@
 			)
 		)
+		(property "Manufacturer" "Microchip Technology"
+			(at 170.18 40.64 0)
+			(effects
+				(font
+					(size 1.27 1.27)
+				)
+				(hide yes)
+			)
+		)
+		(property "MPN" "MIC29302AWD-TR"
+			(at 170.18 40.64 0)
+			(effects
+				(font
+					(size 1.27 1.27)
+				)
+				(hide yes)
+			)
+		)
+		(property "Package" "TO-252-6, DPAK (5 Leads + Tab)"
+			(at 170.18 40.64 0)
+			(effects
+				(font
+					(size 1.27 1.27)
+				)
+				(hide yes)
+			)
+		)
 		(pin "1"
 		)
@@
 			)
 		)
-		(property "MF" "Bosch Sensortec"
+		(property "Manufacturer" "Bosch Sensortec"
 			(at 69.85 105.41 0)
 			(effects
@@
 			)
 		)
-		(property "PACKAGE" "VFLGA-16 Bosch Sensortec"
+		(property "Package" "16-VFLGA Module"
 			(at 69.85 105.41 0)
 			(effects
@@
 			)
 		)
-		(property "MP" "BMI088"
+		(property "MPN" "BMI088"
 			(at 69.85 105.41 0)
 			(effects
@@
 			)
 		)
-		(property "Mouser Part Number" "438-MMC5983MA"
+		(property "MPN" "MMC5983MA"
 			(at 83.82 649.86 0)
 			(effects
@@
 			)
 		)
-		(property "Manufacturer_Name" "MEMSIC"
+		(property "Manufacturer" "MEMSIC"
 			(at 83.82 849.86 0)
 			(effects
@@
 			)
 		)
-		(property "Manufacturer_Part_Number" "MMC5983MA"
-			(at 83.82 949.86 0)
+		(property "Package" "16-VFLGA"
+			(at 46.99 172.72 0)
 			(effects
 				(font
 					(size 1.27 1.27)
 				)
-				(justify left top)
 				(hide yes)
 			)
@@
 			(at 64.77 247.65 0)
 			(effects
+				(font
+					(size 1.27 1.27)
+				)
+				(hide yes)
+			)
+		)
+		(property "Manufacturer" "u-blox"
+			(at 64.77 247.65 0)
+			(effects
+				(font
+					(size 1.27 1.27)
+				)
+				(hide yes)
+			)
+		)
+		(property "MPN" "MAX-M10S-00B"
+			(at 64.77 247.65 0)
+			(effects
+				(font
+					(size 1.27 1.27)
+				)
+				(hide yes)
+			)
+		)
+		(property "Package" "18-SMD Module"
+			(at 64.77 247.65 0)
+			(effects

Commit message: 2025 FINAL
Parts:
- removed IC1: MMC5983MA, HPRfootprints:MMC5983MA_MEM, symbol HPRsymbols:MMC5983MA
- removed J1, J2: Screw_Terminal_01x02, TerminalBlock_TE-Connectivity:TerminalBlock_TE_282834-2_1x02_P2.54mm_Horizontal, symbol Connector:Screw_Terminal_01x02
- removed S1, S2: TS04-66-70-BK-160-SMT, HPRfootprints:SW_TS04-66-70-BK-160-SMT, symbol HPRsymbols:TS04-66-70-BK-160-SMT
- removed U4: MIC29302AWD, Package_TO_SOT_SMD:TO-252-5_TabPin3, symbol Regulator_Linear:MIC29302AWD
- added C11: 100nF, Capacitor_SMD:C_0402_1005Metric_Pad0.74x0.62mm_HandSolder, symbol Device:C
- added J1, J2: 282837-2, HPRfootprints:TE_282837-2, symbol HPRsymbols:282837-2
- added J10, J11: Conn_01x01, Connector_PinHeader_2.54mm:PinHeader_1x01_P2.54mm_Vertical, symbol Connector_Generic:Conn_01x01
- added J12, J13: Conn_Coaxial, Connector_Coaxial:U.FL_Hirose_U.FL-R-SMT-1_Vertical, symbol Connector:Conn_Coaxial
- added J3, J4: Conn_01x03, Connector_PinHeader_2.54mm:PinHeader_1x03_P2.54mm_Vertical, symbol Connector_Generic:Conn_01x03
- added S1, S2: KMR221GLFS, HPRfootprints:SW_KMR221GLFS, symbol HPRsymbols:KMR221GLFS
- added TP4, TP5, TP6, TP7: TestPoint, TestPoint:TestPoint_Pad_1.0x1.0mm, symbol Connector:TestPoint
- added U8: LIS2MDLTR, HPRfootprints:PQFN50P200X200X70-12N, symbol HPRsymbols:LIS2MDLTR
- added U9: MIC29302AWD-TR, HPRfootprints:TO-252-5_MCH, symbol HPRsymbols:MIC29302AWD-TR
- BZ1: MPN (none) -> AT-0927-TT-6-R; Manufacturer (none) -> PUI Audio; Package (none) -> THT; now not fitted
- C1, C3, C4, C5: footprint Capacitor_SMD:C_0201_0603Metric_Pad0.64x0.40mm_HandSolder -> Capacitor_SMD:C_0402_1005Metric_Pad0.74x0.62mm_HandSolder
- C10, C6, C7, C8, C9: footprint Capacitor_SMD:C_0201_0603Metric_Pad0.64x0.40mm_HandSolder -> Capacitor_SMD:C_0603_1608Metric_Pad1.08x0.95mm_HandSolder
- C2: value 1uF -> 220nF; footprint Capacitor_SMD:C_0201_0603Metric_Pad0.64x0.40mm_HandSolder -> Capacitor_SMD:C_0402_1005Metric_Pad0.74x0.62mm_HandSolder
- D1, D2, D3: footprint LED_SMD:LED_0201_0603Metric_Pad0.64x0.40mm_HandSolder -> LED_SMD:LED_0603_1608Metric_Pad1.05x0.95mm_HandSolder
- J5: footprint Connector_JST:JST_XA_B02B-XASK-1-A_1x02_P2.50mm_Vertical -> Connector_JST:JST_PH_S2B-PH-K_1x02_P2.00mm_Horizontal
- J6, J7, M1, M2, TP2, TP3: now not fitted
- J8, J9: MPN (none) -> 132134; Manufacturer (none) -> Amphenol RF; Package (none) -> THT
- Q2: MPN (none) -> MMBT3904LT3G; Package (none) -> SOT-23-3 (TO-236)
- R1, R10, R11, R14, R15, R2, R3, R4, R7, R8, R9: footprint Resistor_SMD:R_0201_0603Metric_Pad0.64x0.40mm_HandSolder -> Resistor_SMD:R_0603_1608Metric_Pad0.98x0.95mm_HandSolder
- TP1: footprint Connector_PinHeader_2.54mm:PinHeader_1x01_P2.54mm_Vertical -> TestPoint:TestPoint_Pad_1.0x1.0mm
- U3: AVAILABILITY In Stock -> (none); DESCRIPTION Accelerometer, Gyroscope, 6 Axis Sensor I²C, SPI Output -> (none); PRICE None -> (none); PURCHASE-URL https://pricing.snapeda.com/search/part/BMI088/?ref=eda -> (none)
Connections:
- net GND: now also R14.2, C11.2, J1.2, J11.1 (Pin_1), J12.2 (Ext), J13.2 (Ext), J2.2, S1.2, S1.5, S2.2, S2.5, U8.6 (GND), U8.8 (GND__1), U9.3 (GND), U9.6 (GND); no longer R15.2
- net SENSE_miso: now also U8.7 (INT/DRDY/SDO)
- net SENSE_mosi: now also U8.4 (SDA/SDI/SDO)
- net SENSE_sck: now also U8.1 (SCL/SPC)
- net VBATT: now also J10.1 (Pin_1), U9.1 (EN), U9.2 (IN)
- net ldo_5v: now also J4.1 (Pin_1), J4.2 (Pin_2), J4.3 (Pin_3)
- net ldo_6v: now also R15.2, U9.4 (OUT); no longer R14.2
- net mag_cs: now also U8.3 (CS)
- net teensy_3.3v: now also C3.1, C11.1, J3.1 (Pin_1), J3.2 (Pin_2), J3.3 (Pin_3), U8.10 (VDD_IO), U8.9 (VDD); no longer C2.1
- net teensy_onoff: now also S2.1
- net at U1.53 (PROGRAM): now also S1.1
- net at J9.1 (In), U6.9 (ANT): now also J13.1 (In)
- net at Q2.1 (B), R2.2: now also TP5.1
- net at Q1.5 (D2_1), Q1.6 (D2_2): now also J2.1, TP7.1
- net at Q1.7 (D1_1), Q1.8 (D1_2): now also J1.1, TP6.1
- net at J8.1 (In), U5.11 (RF_IN): now also J12.1 (In)
- net at R14.1, R15.1: now also U9.5 (ADJ)
- net at Q3.1 (B), R4.2: now also TP4.1
- net mag_int renamed FREE2
- new net: C2.1, U8.5 (C1)
- no-connect marks 14 -> 11
Other:
- moved on the sheet: C2, C3, C8, C9, J8, R14, R15, R7, R8, U5
